Commit message: cambios en robot.urdf.xacro para incluir propiedades y core

File: description/robot.urdf.xacro (robot description, xacro)
@@ -3,5 +3,5 @@
     <!-- Example link -->
     <xacro:include filename="robot_core.xacro"/>
+    <xacro:include filename="properties.urdf.xacro"/>
         <!-- Example link -->
-    <link name="base_link"></link>
 </robot>

Commit message: Cambios de la parte 2

File: description/robot.urdf.xacro (robot description, xacro)
@@ -4,4 +4,5 @@
     <xacro:include filename="robot_core.xacro"/>
     <xacro:include filename="properties.urdf.xacro"/>
+    <xacro:include filename="gazebo_control.xacro"/>
         <!-- Example link -->
 </robot>

File: description/robot_core.xacro (robot description, xacro)
@@ -1,4 +1,18 @@
 <?xml version="1.0"?>
 <robot xmlns:xacro="http://www.ros.org/wiki/xacro">
+    <gazebo reference="chassis">
+        <material>Gazebo/White</material>
+    </gazebo>
+    <gazebo reference="left_wheel">
+        <material>Gazebo/Blue</material>
+    </gazebo>
+    <gazebo reference="right_wheel">
+        <material>Gazebo/Blue</material>
+    </gazebo>
+    <gazebo reference="caster_wheel">
+        <material>Gazebo/Black</material>
+        <mu1 value = "0.001" />
+        <mu2 value = "0.001" />
+    </gazebo>
     <!-- Example link -->
     <xacro:include filename="inertial_macros.xacro"/>

Commit message: lol

File: description/robot.urdf.xacro (robot description, xacro)
@@ -3,6 +3,8 @@
     <!-- Example link -->
     <xacro:include filename="robot_core.xacro"/>
-    <xacro:include filename="properties.urdf.xacro"/>
+    <xacro:include filename="properties.xacro"/>
     <xacro:include filename="gazebo_control.xacro"/>
+    <xacro:include filename="lidar.xacro"/>
+    <xacro:include filename="imu.urdf.xacro"/>
         <!-- Example link -->
 </robot>

File: description/robot_core.xacro (robot description, xacro)
@@ -67,4 +67,9 @@
             <origin xyz="0 0 0" rpy="0 0 0"/>
         </xacro:inertial_cylinder>
+        <collision>
+            <geometry>
+                <sphere radius="0.05"/>
+            </geometry>
+        </collision>
     </link>
     <!-- right wheel joint -->
@@ -91,4 +96,9 @@
             <origin xyz="0 0 0" rpy="0 0 0"/>
         </xacro:inertial_cylinder>
+        <collision>
+            <geometry>
+                <sphere radius="0.05"/>
+            </geometry>
+        </collision>
     </link>
     <!-- caster wheel joint -->
